Commit message: small change

File: lbr_arithmetic_average_roughness/urdf/dummy_robot.urdf (robot description, URDF)
Before this commit: robot dummy_robot, 2 links, 1 joints
Joints:
- joint base_to_camera: origin xyz=0 0 0.3 rpy=0 0.785 0 -> xyz=0 0 0.3 rpy=0 0.700 0

Commit message: implement slope angle analysis

File: lbr_arithmetic_average_roughness/urdf/dummy_robot.urdf (robot description, URDF)
Before this commit: robot dummy_robot, 2 links, 1 joints
Links:
- added link world_frame
Joints:
- added joint world_to_base: type fixed, parent world_frame, child base_link, origin xyz=0 0 0 rpy=0 0 0
